File: PeripheralSOMBreakoutPCB.kicad_sch (KiCad schematic)
At the start: 9 parts, among them J1 Conn_01x02, J2 Conn_01x02, J3 Conn_01x02, J4 Conn_01x02, J5 Conn_01x04, J6 Conn_01x04, J7 Conn_01x01, J8 Conn_01x01

Commit message: board
Parts:
- added J10, J9: CANConnector, UTSVT_Connectors:Molex_MicroFit3.0_1x4xP3.00mm_PolarizingPeg_Vertical, symbol utsvt-connectors:CANConnector
- U1: value ~ -> PeripheralSOM; P/N 53307-2071 -> 53307-2471
Connections:
- new net +12V: J10.1 (5V), J9.1 (5V), U1.22 (+12V_In)
- new net CAN_H: J10.3 (CAN_H), J9.3 (CAN_H), U1.23 (CAN_H)
- new net CAN_L: J10.4 (CAN_L), J9.4 (CAN_L), U1.21 (CAN_L)
- new net GNDPWR: J10.2 (GND), J9.2 (GND), U1.24 (GNDPWR)
